File: ePap.kicad_pcb (KiCad board)
At the start: 2 copper layers, 37.3 x 29.2 mm, 29 parts, among them J1 Conn_01x08, J2 Conn_01x03, J3 Conn_01x02, J4 Conn_01x08, J5 Conn_01x24, J6 Conn_01x34, Q1 Q_NMOS_GSD, U1 AZ1117-3.3

Commit message: V0.2
Parts:
- R1, R2: footprint Resistor_SMD:R_0805_2012Metric_Pad1.15x1.40mm_HandSolder -> Resistor_SMD:R_0603_1608Metric_Pad1.05x0.95mm_HandSolder
- moved C9 6.78 mm to (113.8, 89.4)
- moved R2 0.51 mm to (111.3, 89.4)
- moved R1 0.51 mm to (108.2, 89.4)
- moved J1 0.38 mm to (130.9, 97.5), turned to 270 degrees
Connections:
- J1 pad 1: /VIN -> /BUSY
- J1 pad 2: GND -> /RST
- J1 pad 3: /MOSI -> /D\C
- J1 pad 4: /SCK -> /CS
- J1 pad 5: /CS -> /SCK
- J1 pad 6: /D\C -> /MOSI
- J1 pad 7: /RST -> GND
- J1 pad 8: /BUSY -> /VIN
- U1 pad 4: +3V3 -> (no net)
Routing:
- net /VIN: track 33.1 -> 36.5 mm
- net /CS: track 37.3 -> 40.6 mm
- net /SCK: track 36.6 -> 39.7 mm
- net /RST: track 41.3 -> 44.3 mm
- net /MOSI: track 38.3 -> 41.4 mm
- net /D\C: track 38.5 -> 41.6 mm
- net /BUSY: track 43.7 -> 46.7 mm
- net +3V3: track 51.8 -> 54.0 mm
- net /GDR: track 18.2 -> 19.9 mm
