File: ePap.sch (KiCad schematic (older format))
At the start: 29 parts, among them J1 Conn_01x08, J2 Conn_01x03, J3 Conn_01x02, J4 Conn_01x08, J5 Conn_01x24, J6 Conn_01x34, Q1 Q_NMOS_GSD, U1 AZ1117-3.3

Commit message: V0.2
Connections:
- net BUSY: now also J1.1 (Pin_1); no longer J1.8 (Pin_8)
- net CS: now also J1.4 (Pin_4); no longer J1.5 (Pin_5)
- net D\C: now also J1.3 (Pin_3); no longer J1.6 (Pin_6)
- net GND: now also J1.7 (Pin_7); no longer J1.2 (Pin_2)
- net MOSI: now also J1.6 (Pin_6); no longer J1.3 (Pin_3)
- net RST: now also J1.2 (Pin_2); no longer J1.7 (Pin_7)
- net SCK: now also J1.5 (Pin_5); no longer J1.4 (Pin_4)
- net VIN: now also J1.8 (Pin_8); no longer J1.1 (Pin_1)
Changed lines of the file:
@@
 L Connector_Generic:Conn_01x08 J1
 U 1 1 5EC8F581
-P 1250 1800
-F 0 "J1" H 1168 2317 50  0000 C CNN
-F 1 "Conn_01x08" H 1168 2226 50  0000 C CNN
-F 2 "Connector_FFC-FPC:TE_0-1734839-8_1x08-1MP_P0.5mm_Horizontal" H 1250 1800 50  0001 C CNN
-F 3 "~" H 1250 1800 50  0001 C CNN
-	1    1250 1800
-	-1   0    0    -1
+P 1250 1900
+F 0 "J1" H 1168 2417 50  0000 C CNN
+F 1 "Conn_01x08" H 1168 2326 50  0000 C CNN
+F 2 "Connector_FFC-FPC:TE_0-1734839-8_1x08-1MP_P0.5mm_Horizontal" H 1250 1900 50  0001 C CNN
+F 3 "~" H 1250 1900 50  0001 C CNN
+	1    1250 1900
+	-1   0    0    1
 $EndComp
 Wire Wire Line
